Commit message: 添加夹爪 + 场景目标

File: src/armpy_description/urdf/simple_arm.urdf.xacro (robot description, xacro)
@@ -3,4 +3,5 @@
   <xacro:property name="upper_len" value="0.22"/>
   <xacro:property name="forearm_len" value="0.18"/>
+  <xacro:property name="finger_len" value="0.08"/>
   <material name="dark_gray">
     <color rgba="0.18 0.20 0.22 1.0"/>
@@ -88,16 +89,46 @@
     </visual>
   </link>
-  <joint name="gripper_joint" type="revolute">
+  <joint name="gripper_mount_joint" type="fixed">
     <parent link="wrist_link"/>
-    <child link="gripper_link"/>
+    <child link="gripper_palm"/>
     <origin xyz="0.05 0 0" rpy="0 0 0"/>
-    <axis xyz="1 0 0"/>
-    <limit lower="-0.4" upper="0.4" effort="1" velocity="1"/>
   </joint>
-  <link name="gripper_link">
+  <link name="gripper_palm">
     <visual>
-      <origin xyz="0.035 0 0" rpy="0 0 0"/>
+      <origin xyz="0.02 0 0" rpy="0 0 0"/>
       <geometry>
-        <box size="0.07 0.06 0.018"/>
+        <box size="0.04 0.07 0.018"/>
+      </geometry>
+      <material name="dark_gray"/>
+    </visual>
+  </link>
+  <joint name="left_finger_joint" type="prismatic">
+    <parent link="gripper_palm"/>
+    <child link="left_finger"/>
+    <origin xyz="0.04 0.026 0" rpy="0 0 0"/>
+    <axis xyz="0 1 0"/>
+    <limit lower="0.0" upper="0.025" effort="1" velocity="0.1"/>
+  </joint>
+  <link name="left_finger">
+    <visual>
+      <origin xyz="${finger_len / 2} 0 0" rpy="0 0 0"/>
+      <geometry>
+        <box size="${finger_len} 0.012 0.018"/>
+      </geometry>
+      <material name="dark_gray"/>
+    </visual>
+  </link>
+  <joint name="right_finger_joint" type="prismatic">
+    <parent link="gripper_palm"/>
+    <child link="right_finger"/>
+    <origin xyz="0.04 -0.026 0" rpy="0 0 0"/>
+    <axis xyz="0 -1 0"/>
+    <limit lower="0.0" upper="0.025" effort="1" velocity="0.1"/>
+  </joint>
+  <link name="right_finger">
+    <visual>
+      <origin xyz="${finger_len / 2} 0 0" rpy="0 0 0"/>
+      <geometry>
+        <box size="${finger_len} 0.012 0.018"/>
       </geometry>
       <material name="dark_gray"/>
